File: nRF51822.sch (KiCad schematic (older format))
At the start: 26 parts, among them U2 NRF51822, X1 32.768kHz, X2 16Mhz

Commit message: 0.0.2
Parts:
- C10, C11, C12, C13, C14, C15, C16, C17, C18, C19, C20, C21, C7, C8, C9: footprint ~ -> Local:SMD-0402_c
- FB2, FB3, L1, L2, L3, L4: footprint ~ -> Local:SMD-0402
- R1, R2: footprint ~ -> Local:SMD-0402_r
- U2: footprint ~ -> Local:QFN48
- X1: footprint ~ -> (none)
- X2: footprint ~ -> Crystals_Oscillators_SMD:crystal_FA238-TSX3225
Connections:
- net XL1: now also X1.1; no longer X1.2
- net XL2: now also X1.2; no longer X1.1
Changed lines of the file:
@@
 LIBS:adxl362
 LIBS:aux_lcd-cache
-EELAYER 27 0
+EELAYER 24 0
 EELAYER END
 $Descr A4 11693 8268
@@
 $EndDescr
 $Comp
-L CRYSTAL X1
-U 1 1 53233167
-P 7500 2100
-F 0 "X1" H 7500 2250 60  0000 C CNN
-F 1 "32.768kHz" H 7500 1950 40  0000 C CNN
-F 2 "~" H 7500 2100 60  0000 C CNN
-F 3 "~" H 7500 2100 60  0000 C CNN
-	1    7500 2100
-	0    -1   -1   0
-$EndComp
-$Comp
 L C C15
 U 1 1 53233182
@@
 F 0 "C15" H 7800 1900 40  0000 L CNN
 F 1 "12pF" H 7806 1715 40  0000 L CNN
-F 2 "~" H 7838 1650 30  0000 C CNN
+F 2 "Local:SMD-0402_c" H 7838 1650 30  0000 C CNN
 F 3 "~" H 7800 1800 60  0000 C CNN
 	1    7800 1800
@@
 F 0 "C16" H 7800 2500 40  0000 L CNN
 F 1 "12pF" H 7806 2315 40  0000 L CNN
-F 2 "~" H 7838 2250 30  0000 C CNN
+F 2 "Local:SMD-0402_c" H 7838 2250 30  0000 C CNN
 F 3 "~" H 7800 2400 60  0000 C CNN
 	1    7800 2400
@@
 $EndComp
 $Comp
-L GND #PWR04
+L GND #PWR1
 U 1 1 53233229
 P 8000 2550
-F 0 "#PWR04" H 8000 2550 30  0001 C CNN
+F 0 "#PWR1" H 8000 2550 30  0001 C CNN
 F 1 "GND" H 8000 2480 30  0001 C CNN
 F 2 "" H 8000 2550 60  0000 C CNN
@@
 F 0 "X2" H 8550 2250 60  0000 C CNN
 F 1 "16Mhz" H 8550 1950 60  0000 C CNN
-F 2 "~" H 8550 2100 60  0000 C CNN
+F 2 "Crystals_Oscillators_SMD:crystal_FA238-TSX3225" H 8550 2100 60  0000 C CNN
 F 3 "~" H 8550 2100 60  0000 C CNN
 	1    8550 2100
@@
 F 0 "C19" H 8850 1900 40  0000 L CNN
 F 1 "12pF" H 8856 1715 40  0000 L CNN
-F 2 "~" H 8888 1650 30  0000 C CNN
+F 2 "Local:SMD-0402_c" H 8888 1650 30  0000 C CNN
 F 3 "~" H 8850 1800 60  0000 C CNN
 	1    8850 1800
@@
 F 0 "C20" H 8850 2500 40  0000 L CNN
 F 1 "12pF" H 8856 2315 40  0000 L CNN
-F 2 "~" H 8888 2250 30  0000 C CNN
+F 2 "Local:SMD-0402_c" H 8888 2250 30  0000 C CNN
 F 3 "~" H 8850 2400 60  0000 C CNN
 	1    8850 2400
@@
 $EndComp
 $Comp
-L GND #PWR05
+L GND #PWR2
 U 1 1 53233299
 P 9050 2550
-F 0 "#PWR05" H 9050 2550 30  0001 C CNN
+F 0 "#PWR2" H 9050 2550 30  0001 C CNN
 F 1 "GND" H 9050 2480 30  0001 C CNN
 F 2 "" H 9050 2550 60  0000 C CNN
@@
 F 0 "U2" H 5050 3550 60  0000 C CNN
 F 1 "NRF51822" H 5050 3900 60  0000 C CNN
-F 2 "~" H 5050 3700 60  0000 C CNN
+F 2 "Local:QFN48" H 5050 3700 60  0000 C CNN
 F 3 "~" H 5050 3700 60  0000 C CNN
 	1    5050 3700
@@
 F 0 "C8" H 3150 4850 40  0000 L CNN
 F 1 "100nF" H 3156 4665 40  0000 L CNN
-F 2 "~" H 3188 4600 30  0000 C CNN
+F 2 "Local:SMD-0402_c" H 3188 4600 30  0000 C CNN
 F 3 "~" H 3150 4750 60  0000 C CNN
 	1    3150 4750
@@
 F 0 "C9" H 3400 4850 40  0000 L CNN
 F 1 "4.7µF" H 3406 4665 40  0000 L CNN
-F 2 "~" H 3438 4600 30  0000 C CNN
+F 2 "Local:SMD-0402_c" H 3438 4600 30  0000 C CNN
 F 3 "~" H 3400 4750 60  0000 C CNN
 	1    3400 4750
@@
 F 0 "C10" H 3650 4850 40  0000 L CNN
 F 1 "100nF" H 3656 4665 40  0000 L CNN
-F 2 "~" H 3688 4600 30  0000 C CNN
+F 2 "Local:SMD-0402_c" H 3688 4600 30  0000 C CNN
 F 3 "~" H 3650 4750 60  0000 C CNN
 	1    3650 4750
@@
 F 0 "R1" V 6030 4850 40  0000 C CNN
 F 1 "12k" V 5957 4851 40  0000 C CNN
-F 2 "~" V 5880 4850 30  0000 C CNN
+F 2 "Local:SMD-0402_r" V 5880 4850 30  0000 C CNN
 F 3 "~" H 5950 4850 30  0000 C CNN
 	1    5950 4850
@@
 F 0 "C11" H 6800 3400 40  0000 L CNN
 F 1 "1nF" H 6806 3215 40  0000 L CNN
-F 2 "~" H 6838 3150 30  0000 C CNN
+F 2 "Local:SMD-0402_c" H 6838 3150 30  0000 C CNN
 F 3 "~" H 6800 3300 60  0000 C CNN
 	1    6800 3300
@@
 F 0 "C12" H 6800 4850 40  0000 L CNN
 F 1 "47nF" H 6806 4665 40  0000 L CNN
-F 2 "~" H 6838 4600 30  0000 C CNN
+F 2 "Local:SMD-0402_c" H 6838 4600 30  0000 C CNN
 F 3 "~" H 6800 4750 60  0000 C CNN
 	1    6800 4750
@@
 F 0 "C13" H 7200 4850 40  0000 L CNN
 F 1 "2.2nF" H 7206 4665 40  0000 L CNN
-F 2 "~" H 7238 4600 30  0000 C CNN
+F 2 "Local:SMD-0402_c" H 7238 4600 30  0000 C CNN
 F 3 "~" H 7200 4750 60  0000 C CNN
 	1    7200 4750
@@
 F 0 "C18" H 8700 3750 40  0000 L CNN
 F 1 "1.5pF" H 8706 3565 40  0000 L CNN
-F 2 "~" H 8738 3500 30  0000 C CNN
+F 2 "Local:SMD-0402_c" H 8738 3500 30  0000 C CNN
 F 3 "~" H 8700 3650 60  0000 C CNN
 	1    8700 3650
@@
 F 0 "C21" H 8950 3750 40  0000 L CNN
 F 1 "1pF" H 8956 3565 40  0000 L CNN
-F 2 "~" H 8988 3500 30  0000 C CNN
+F 2 "Local:SMD-0402_c" H 8988 3500 30  0000 C CNN
 F 3 "~" H 8950 3650 60  0000 C CNN
 	1    8950 3650
@@
 F 0 "C14" H 7600 3100 40  0000 L CNN
 F 1 "2.2pF" H 7606 2915 40  0000 L CNN
-F 2 "~" H 7638 2850 30  0000 C CNN
+F 2 "Local:SMD-0402_c" H 7638 2850 30  0000 C CNN
 F 3 "~" H 7600 3000 60  0000 C CNN
 	1    7600 3000
@@
 F 0 "R2" V 9380 3000 40  0000 C CNN
 F 1 "0" V 9307 3001 40  0000 C CNN
-F 2 "~" V 9230 3000 30  0000 C CNN
+F 2 "Local:SMD-0402_r" V 9230 3000 30  0000 C CNN
 F 3 "~" H 9300 3000 30  0000 C CNN
 	1    9300 3000
@@
 F 0 "L2" V 7150 4000 40  0000 C CNN
 F 1 "10nH" V 7300 4000 40  0000 C CNN
-F 2 "~" H 7200 4000 60  0000 C CNN
+F 2 "Local:SMD-0402" H 7200 4000 60  0000 C CNN
 F 3 "~" H 7200 4000 60  0000 C CNN
 	1    7200 4000
@@
 F 0 "L1" V 7150 3300 40  0000 C CNN
 F 1 "4.7nH" V 7300 3300 40  0000 C CNN
-F 2 "~" H 7200 3300 60  0000 C CNN
+F 2 "Local:SMD-0402" H 7200 3300 60  0000 C CNN
 F 3 "~" H 7200 3300 60  0000 C CNN
 	1    7200 3300
@@
 F 0 "L3" V 8250 3000 40  0000 C CNN
 F 1 "3.3nH" V 8400 3000 40  0000 C CNN
-F 2 "~" H 8300 3000 60  0000 C CNN
+F 2 "Local:SMD-0402" H 8300 3000 60  0000 C CNN
 F 3 "~" H 8300 3000 60  0000 C CNN
 	1    8300 3000
@@
 F 0 "L4" V 9600 3650 40  0000 C CNN
 F 1 "1.8nH" V 9750 3650 40  0000 C CNN
-F 2 "~" H 9650 3650 60  0000 C CNN
+F 2 "Local:SMD-0402" H 9650 3650 60  0000 C CNN
 F 3 "~" H 9650 3650 60  0000 C CNN
 	1    9650 3650
@@
 F 0 "C17" H 7900 3750 40  0000 L CNN
 F 1 "0.8pF" H 7906 3565 40  0000 L CNN
-F 2 "~" H 7938 3500 30  0000 C CNN
+F 2 "Local:SMD-0402_c" H 7938 3500 30  0000 C CNN
 F 3 "~" H 7900 3650 60  0000 C CNN
 	1    7900 3650
@@
 F 0 "FB3" H 2700 3400 60  0000 C CNN
 F 1 "10µH" H 2700 3150 60  0000 C CNN
-F 2 "~" H 2700 3250 60  0000 C CNN
+F 2 "Local:SMD-0402" H 2700 3250 60  0000 C CNN
 F 3 "~" H 2700 3250 60  0000 C CNN
 	1    2700 3250
@@
 F 0 "FB2" H 1950 3400 60  0000 C CNN
 F 1 "15nH" H 1950 3150 60  0000 C CNN
-F 2 "~" H 1950 3250 60  0000 C CNN
+F 2 "Local:SMD-0402" H 1950 3250 60  0000 C CNN
 F 3 "~" H 1950 3250 60  0000 C CNN
 	1    1950 3250
@@
 F 0 "C7" H 1600 4850 40  0000 L CNN
 F 1 "1µF" H 1606 4665 40  0000 L CNN
-F 2 "~" H 1638 4600 30  0000 C CNN
+F 2 "Local:SMD-0402_c" H 1638 4600 30  0000 C CNN
 F 3 "~" H 1600 4750 60  0000 C CNN
 	1    1600 4750
@@
 Connection ~ 3650 4250
 $Comp
-L PWR_FLAG #FLG06
+L PWR_FLAG #FLG4
 U 1 1 532A1CFA
 P 1600 3250
-F 0 "#FLG06" H 1600 3345 30  0001 C CNN
+F 0 "#FLG4" H 1600 3345 30  0001 C CNN
 F 1 "PWR_FLAG" H 1600 3430 30  0000 C CNN
 F 2 "" H 1600 3250 60  0000 C CNN
@@
 	0    -1   -1   0
 $EndComp
+$Comp
+L CRYSTAL X1
+U 1 1 54020623
+P 7500 2100
+F 0 "X1" H 7500 2250 60  0000 C CNN
+F 1 "32.768kHz" H 7500 1950 60  0000 C CNN
+F 2 "" H 7500 2100 60  0000 C CNN
+F 3 "" H 7500 2100 60  0000 C CNN
+	1    7500 2100
+	0    1    1    0
+$EndComp
 $EndSCHEMATC
